File: Electronics/ProtoRev0/BrailleBoy/FETsDrivers.sch (KiCad schematic (older format))
At the start: 43 parts, among them Q10 L1, Q11 L2, Q12 L3, Q13 L4, Q14 L5, Q3 H0, Q4 H1, Q5 H2, Q6 H3, Q7 H4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

Commit message: Added some annotations to make things rather professional :)
Parts:
- C18: renamed from C20; footprint Capacitors_SMD:C_0805 -> (none)
- C19: renamed from C21; footprint Capacitors_SMD:C_0805 -> (none)
- C20: renamed from C22; footprint Capacitors_SMD:C_0805 -> (none)
- C21: renamed from C23; footprint Capacitors_SMD:C_0805 -> (none)
- C22: renamed from C24; footprint Capacitors_SMD:C_0805 -> (none)
- C23: renamed from C25; footprint Capacitors_SMD:C_0805 -> (none)
- R23: renamed from R24; footprint Resistors_SMD:R_0805 -> (none)
- R24: renamed from R23; footprint Resistors_SMD:R_0805 -> (none)
- R25: renamed from R26; footprint Resistors_SMD:R_0805 -> (none)
- R26: renamed from R25; footprint Resistors_SMD:R_0805 -> (none)
- R27, R28, R29, R30, R31, R32, R33, R34: footprint Resistors_SMD:R_0805 -> (none)
- U10, U11, U12, U13, U14, U15, U16, U17, U18, U7, U8, U9: footprint Housings_SSOP:TSOP-6_1.65x3.05mm_Pitch0.95mm -> (none)
- U19: footprint TO_SOT_Packages_SMD:SOT-23-6 -> (none)
