File: Electronics/ProtoRev0/BrailleBoy/FETsDrivers.sch (KiCad schematic (older format))
At the start: 43 parts, among them Q3 H0, Q9 L0, U10 PMD3001D, U11 PMD3001D, U12 PMD3001D, U13 PMD3001D, U14 PMD3001D, U15 PMD3001D, U16 PMD3001D, U17 PMD3001D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

Commit message: Made the schematic sheets a bit prettier
Parts:
- C18, C19, C20, C21, C22, C23: footprint (none) -> Capacitors_SMD:C_0805
- gave numbers to parts that had none: 10
Changed lines of the file:
@@
 F 0 "C18" V 8500 2800 50  0000 C CNN
 F 1 "0.1uF" V 8650 2750 50  0000 C CNN
-F 2 "" H 8550 2750 50  0001 C CNN
+F 2 "Capacitors_SMD:C_0805" H 8550 2750 50  0001 C CNN
 F 3 "" H 8550 2750 50  0001 C CNN
 	1    8550 2750
@@
 F 0 "C20" V 9250 2950 50  0000 C CNN
 F 1 "0.1uF" V 9100 3050 50  0000 C CNN
-F 2 "" H 9200 3050 50  0001 C CNN
+F 2 "Capacitors_SMD:C_0805" H 9200 3050 50  0001 C CNN
 F 3 "" H 9200 3050 50  0001 C CNN
 	1    9200 3050
@@
 F 0 "C21" V 9150 3350 50  0000 C CNN
 F 1 "10uF" V 9300 3250 50  0000 C CNN
-F 2 "" H 9200 3250 50  0001 C CNN
+F 2 "Capacitors_SMD:C_0805" H 9200 3250 50  0001 C CNN
 F 3 "" H 9200 3250 50  0001 C CNN
 	1    9200 3250
@@
 F 0 "C19" V 8500 3000 50  0000 C CNN
 F 1 "10uF" V 8650 2950 50  0000 C CNN
-F 2 "" H 8550 2950 50  0001 C CNN
+F 2 "Capacitors_SMD:C_0805" H 8550 2950 50  0001 C CNN
 F 3 "" H 8550 2950 50  0001 C CNN
 	1    8550 2950
@@
 F 0 "C22" H 9900 2650 50  0000 L CNN
 F 1 "0.1uF" H 9900 2500 50  0000 L CNN
-F 2 "" H 9900 2600 50  0001 C CNN
+F 2 "Capacitors_SMD:C_0805" H 9900 2600 50  0001 C CNN
 F 3 "" H 9900 2600 50  0001 C CNN
 	1    9900 2600
@@
 F 0 "C23" H 10100 2650 50  0000 L CNN
 F 1 "10uF" H 10100 2550 50  0000 L CNN
-F 2 "" H 10100 2600 50  0001 C CNN
+F 2 "Capacitors_SMD:C_0805" H 10100 2600 50  0001 C CNN
 F 3 "" H 10100 2600 50  0001 C CNN
 	1    10100 2600
@@
 AR Path="/5BAEF395" Ref="Q?"  Part="1"
 AR Path="/5B7BE201/5BAEF395" Ref="Q?"  Part="1"
-AR Path="/5B7BE201/5C1CF809/5BAEF395" Ref="Q?"  Part="1"
-F 0 "Q?" H 5956 1496 50  0000 L CNN
+AR Path="/5B7BE201/5C1CF809/5BAEF395" Ref="Q10"  Part="1"
+F 0 "Q10" H 5956 1496 50  0000 L CNN
 F 1 "L0" H 5956 1405 50  0000 L CNN
 F 2 "" H 5950 1550 50  0001 C CNN
@@
 AR Path="/5BAEF40D" Ref="Q?"  Part="1"
 AR Path="/5B7BE201/5BAEF40D" Ref="Q?"  Part="1"
-AR Path="/5B7BE201/5C1CF809/5BAEF40D" Ref="Q?"  Part="1"
-F 0 "Q?" H 6656 1496 50  0000 L CNN
+AR Path="/5B7BE201/5C1CF809/5BAEF40D" Ref="Q11"  Part="1"
+F 0 "Q11" H 6656 1496 50  0000 L CNN
 F 1 "L0" H 6656 1405 50  0000 L CNN
 F 2 "" H 6650 1550 50  0001 C CNN
@@
 AR Path="/5BAEF487" Ref="Q?"  Part="1"
 AR Path="/5B7BE201/5BAEF487" Ref="Q?"  Part="1"
-AR Path="/5B7BE201/5C1CF809/5BAEF487" Ref="Q?"  Part="1"
-F 0 "Q?" H 7356 1496 50  0000 L CNN
+AR Path="/5B7BE201/5C1CF809/5BAEF487" Ref="Q12"  Part="1"
+F 0 "Q12" H 7356 1496 50  0000 L CNN
 F 1 "L0" H 7356 1405 50  0000 L CNN
 F 2 "" H 7350 1550 50  0001 C CNN
@@
 AR Path="/5BAEF503" Ref="Q?"  Part="1"
 AR Path="/5B7BE201/5BAEF503" Ref="Q?"  Part="1"
-AR Path="/5B7BE201/5C1CF809/5BAEF503" Ref="Q?"  Part="1"
-F 0 "Q?" H 8006 1496 50  0000 L CNN
+AR Path="/5B7BE201/5C1CF809/5BAEF503" Ref="Q13"  Part="1"
+F 0 "Q13" H 8006 1496 50  0000 L CNN
 F 1 "L0" H 8006 1405 50  0000 L CNN
 F 2 "" H 8000 1550 50  0001 C CNN
@@
 AR Path="/5BAEF57F" Ref="Q?"  Part="1"
 AR Path="/5B7BE201/5BAEF57F" Ref="Q?"  Part="1"
-AR Path="/5B7BE201/5C1CF809/5BAEF57F" Ref="Q?"  Part="1"
-F 0 "Q?" H 8656 1496 50  0000 L CNN
+AR Path="/5B7BE201/5C1CF809/5BAEF57F" Ref="Q14"  Part="1"
+F 0 "Q14" H 8656 1496 50  0000 L CNN
 F 1 "L0" H 8656 1405 50  0000 L CNN
 F 2 "" H 8650 1550 50  0001 C CNN
@@
 P 1650 1250
 AR Path="/5B7BE201/5BAF06CE" Ref="Q?"  Part="1"
-AR Path="/5B7BE201/5C1CF809/5BAF06CE" Ref="Q?"  Part="1"
-F 0 "Q?" H 1856 1204 50  0000 L CNN
+AR Path="/5B7BE201/5C1CF809/5BAF06CE" Ref="Q4"  Part="1"
+F 0 "Q4" H 1856 1204 50  0000 L CNN
 F 1 "H0" H 1856 1295 50  0000 L CNN
 F 2 "" H 1850 1350 50  0001 C CNN
@@
 P 2350 1250
 AR Path="/5B7BE201/5BAF074A" Ref="Q?"  Part="1"
-AR Path="/5B7BE201/5C1CF809/5BAF074A" Ref="Q?"  Part="1"
-F 0 "Q?" H 2556 1204 50  0000 L CNN
+AR Path="/5B7BE201/5C1CF809/5BAF074A" Ref="Q5"  Part="1"
+F 0 "Q5" H 2556 1204 50  0000 L CNN
 F 1 "H0" H 2556 1295 50  0000 L CNN
 F 2 "" H 2550 1350 50  0001 C CNN
@@
 P 3050 1250
 AR Path="/5B7BE201/5BAF07C8" Ref="Q?"  Part="1"
-AR Path="/5B7BE201/5C1CF809/5BAF07C8" Ref="Q?"  Part="1"
-F 0 "Q?" H 3256 1204 50  0000 L CNN
+AR Path="/5B7BE201/5C1CF809/5BAF07C8" Ref="Q6"  Part="1"
+F 0 "Q6" H 3256 1204 50  0000 L CNN
 F 1 "H0" H 3256 1295 50  0000 L CNN
 F 2 "" H 3250 1350 50  0001 C CNN
@@
 P 3700 1250
 AR Path="/5B7BE201/5BAF0844" Ref="Q?"  Part="1"
-AR Path="/5B7BE201/5C1CF809/5BAF0844" Ref="Q?"  Part="1"
-F 0 "Q?" H 3906 1204 50  0000 L CNN
+AR Path="/5B7BE201/5C1CF809/5BAF0844" Ref="Q7"  Part="1"
+F 0 "Q7" H 3906 1204 50  0000 L CNN
 F 1 "H0" H 3906 1295 50  0000 L CNN
 F 2 "" H 3900 1350 50  0001 C CNN
@@
 P 4350 1250
 AR Path="/5B7BE201/5BAF08C0" Ref="Q?"  Part="1"
-AR Path="/5B7BE201/5C1CF809/5BAF08C0" Ref="Q?"  Part="1"
-F 0 "Q?" H 4556 1204 50  0000 L CNN
+AR Path="/5B7BE201/5C1CF809/5BAF08C0" Ref="Q8"  Part="1"
+F 0 "Q8" H 4556 1204 50  0000 L CNN
 F 1 "H0" H 4556 1295 50  0000 L CNN
 F 2 "" H 4550 1350 50  0001 C CNN
