File: Electronics/ProtoRev0/BrailleBoy/FETsDrivers.sch (KiCad schematic (older format))
At the start: 43 parts, among them Q10 L0, Q11 L0, Q12 L0, Q13 L0, Q14 L0, Q3 H0, Q4 H0, Q5 H0, Q6 H0, Q7 H0, Q8 H0, Q9 L0, U10 PMD3001D, U11 PMD3001D, U12 PMD3001D, U13 PMD3001D, U14 PMD3001D, U15 PMD3001D, U16 PMD3001D, U17 PMD3001D, U18 PMD3001D, U19 TC1240(A), U7 PMD3001D, U8 PMD3001D, U9 PMD3001D

Commit message: Uploading all files to transfer this project to another team who is interested in continuing it
Parts:
- removed R24, R26, R28, R30, R32, R34: 10K, symbol Device:R
- removed U10, U11, U12, U13, U14, U15, U16, U17, U18, U7, U8, U9: PMD3001D, symbol Custom:PMD3001D
- removed U19: TC1240(A), symbol Custom:TC1240(A)
- added U? (x12): PMD3001D, symbol Custom:PMD3001D
- added U?: TC1240(A), symbol Custom:TC1240(A)
Connections:
- net DRIVER_VOLTAGE_OUT: now also U?.5 (CollectorTR1), U?.5 (CollectorTR1), U?.5 (CollectorTR1), U?.5 (CollectorTR1), U?.5 (CollectorTR1), U?.5 (CollectorTR1), U?.5 (Vout), U?.6 (CollectorTR1), U?.6 (CollectorTR1), U?.6 (CollectorTR1), U?.6 (CollectorTR1), U?.6 (CollectorTR1), U?.6 (CollectorTR1)
- net GROUND_IN: now also U?.2 (Collector_TR2), U?.2 (Collector_TR2), U?.2 (Collector_TR2), U?.2 (Collector_TR2), U?.2 (Collector_TR2), U?.2 (Collector_TR2), U?.2 (Collector_TR2), U?.2 (Collector_TR2), U?.2 (Collector_TR2), U?.2 (Collector_TR2), U?.2 (Collector_TR2), U?.2 (Collector_TR2), U?.2 (GND), U?.3 (Collector_TR2), U?.3 (Collector_TR2), U?.3 (Collector_TR2), U?.3 (Collector_TR2), U?.3 (Collector_TR2), U?.3 (Collector_TR2), U?.3 (Collector_TR2), U?.3 (Collector_TR2), U?.3 (Collector_TR2), U?.3 (Collector_TR2), U?.3 (Collector_TR2), U?.3 (Collector_TR2), U?.4 (SHDN)
- net HIGH0: now also U?.1 (Base_COM)
- net HIGH1: now also U?.1 (Base_COM)
- net HIGH2: now also U?.1 (Base_COM)
- net HIGH3: now also U?.1 (Base_COM)
- net HIGH4: now also U?.1 (Base_COM)
- net HIGH5: now also U?.1 (Base_COM)
- net High0: now also U?.4 (EmitterCom)
- net High1: now also U?.4 (EmitterCom)
- net High2: now also U?.4 (EmitterCom)
- net High3: now also U?.4 (EmitterCom)
- net High4: now also U?.4 (EmitterCom)
- net High5: now also U?.4 (EmitterCom)
- net LOW0: now also U?.1 (Base_COM)
- net LOW1: now also U?.1 (Base_COM)
- net LOW2: now also U?.1 (Base_COM)
- net LOW3: now also U?.1 (Base_COM)
- net LOW4: now also U?.1 (Base_COM)
- net LOW5: now also U?.1 (Base_COM)
- net Low0: now also U?.4 (EmitterCom)
- net Low1: now also U?.4 (EmitterCom)
- net Low2: now also U?.4 (EmitterCom)
- net Low3: now also U?.4 (EmitterCom)
- net Low4: now also U?.4 (EmitterCom)
- net Low5: now also U?.4 (EmitterCom)
- net POWER_IN: now also U?.1 (Vin), U?.5 (CollectorTR1), U?.5 (CollectorTR1), U?.5 (CollectorTR1), U?.5 (CollectorTR1), U?.5 (CollectorTR1), U?.5 (CollectorTR1), U?.6 (CollectorTR1), U?.6 (CollectorTR1), U?.6 (CollectorTR1), U?.6 (CollectorTR1), U?.6 (CollectorTR1), U?.6 (CollectorTR1)
- net at C20.1, C21.2: now also U?.3 (C-)
- net at C20.2, C21.1: now also U?.6 (C+)
