File: Electronics/ProtoRev0/BrailleBoy/BrailleBoy.sch (KiCad schematic (older format))
At the start: 33 parts, among them SW1 B0, SW2 B1, SW3 B2, SW4 B3, SW5 RESET, U1 MCP23S17, U3 ESP32-WROOM

Commit message: Added some annotations to make things rather professional :)
Parts:
- U2: renamed from U?; footprint (none) -> Custom:SPH0645_BRK_Adafruit
- renumbered C8 to C6, C9 to C7, C10 to C8, R6 to R5, R7 to R6, R5 to R7
Other:
- note added: "ESP32 - MAIN SOC"
- moved on the sheet: C1, C2, C3, C4, C5, C6, C7, C8, D1, D2, D3, D4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

Commit message: Made the schematic sheets a bit prettier
Parts:
- renumbered C2 to C1, C3 to C2, C4 to C3, C5 to C4, C1 to C5
Other:
- moved on the sheet: C1, C2, C3, C4, C5, R1, R2, R3, R4, R5, R6, R7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
