File: Electronics/ProtoRev0/BrailleBoy/BrailleBoy.sch (KiCad schematic (older format))
At the start: 33 parts, among them SW1 B0, SW2 B1, SW3 B2, SW4 B3, SW5 RESET, U1 MCP23S17, U2 SPH0645-BRK-ADAFRUIT, U3 ESP32-WROOM

Commit message: Uploading all files to transfer this project to another team who is interested in continuing it
Parts:
- removed U1: MCP23S17, Housings_SOIC:SOIC-16_3.9x9.9mm_Pitch1.27mm, symbol Custom:MCP23S17
- removed U2: SPH0645-BRK-ADAFRUIT, Custom:SPH0645_BRK_Adafruit, symbol Custom:SPH0645-BRK-ADAFRUIT
- removed U3: ESP32-WROOM, ESP32-footprints-Lib:ESP32-WROOM, symbol ESP32-footprints-Shem-Lib:ESP32-WROOM
- added U?: ESP32-WROOM, ESP32-footprints-Lib:ESP32-WROOM, symbol ESP32-footprints-Shem-Lib:ESP32-WROOM
- added U?: MCP23S17, symbol Custom:MCP23S17
- added U?: SPH0645-BRK-ADAFRUIT, symbol Custom:SPH0645-BRK-ADAFRUIT
Connections:
- net +3V3: now also SW1.1, SW2.1, SW3.1, SW4.1, U?.18 (~RESET), U?.2 (3V3), U?.3 (DOUT), U?.9 (VDD); no longer C1.2, C2.1, C3.1, C4.1
- net BatterySense: now also U?.4 (SENSOR_VP)
- net BootOption: now also U?.25 (IO0)
- net Button0: now also U?.6 (IO34)
- net Button1: now also U?.7 (IO35)
- net Button2: now also U?.8 (IO32)
- net Button3: now also U?.9 (IO33)
- net EspRx: now also U?.34 (RXD0)
- net EspTx: now also U?.35 (TXD0)
- net GND: now also C1.2, C2.2, C3.2, C4.2, U?.1 (GND), U?.10 (VSS), U?.15 (A0), U?.15 (GND), U?.16 (A1), U?.17 (A2), U?.2 (LCRL/WS), U?.38 (GND), U?.39 (GND-PAD), U?.4 (BCLK); no longer SW1.1, SW2.1, SW3.1, SW4.1
- net MicBclk: now also U?.11 (IO26)
- net MicData: now also U?.12 (IO27)
- net MicWs: now also U?.10 (IO25)
- net Reset: now also U?.3 (EN)
- net SolenoidFetMatrix/High0: now also U?.21 (GPA0)
- net SolenoidFetMatrix/High1: now also U?.22 (GPA1)
- net SolenoidFetMatrix/High2: now also U?.23 (GPA2)
- net SolenoidFetMatrix/High3: now also U?.24 (GPA3)
- net SolenoidFetMatrix/High4: now also U?.25 (GPA4)
- net SolenoidFetMatrix/High5: now also U?.26 (GPA5)
- net SolenoidFetMatrix/LOW0: now also U?.1 (GPB0)
- net SolenoidFetMatrix/LOW1: now also U?.2 (GPB1)
- net SolenoidFetMatrix/LOW2: now also U?.3 (GPB2)
- net SolenoidFetMatrix/LOW3: now also U?.4 (GPB3)
- net SolenoidFetMatrix/LOW4: now also U?.5 (GPB4)
- net SolenoidFetMatrix/LOW5: now also U?.6 (GPB5)
- net SpiClk: now also U?.12 (SCK), U?.13 (IO14)
- net SpiCs0: now also U?.11 (CS), U?.23 (IO15)
- net SpiMiso: now also U?.14 (IO12), U?.14 (MISO)
- net SpiMosi: now also U?.13 (MOSI), U?.16 (IO13)
- net at D4.1 (K): now also U?.26 (IO4)
- net at D3.1 (K): now also U?.29 (IO5)
- net at D2.1 (K): now also U?.30 (IO18)
- net at D1.1 (K): now also U?.31 (IO19)
- net at R6.2: now also U?.6 (3V3)
- net at R5.2: now also U?.1 (SEL)
- net at R7.2: now also U?.5 (GND)
- net at R2.1, SW2.2: now also C2.1; no longer C2.2
- net at R3.1, SW3.2: now also C3.1; no longer C3.2
- net at R4.1, SW4.2: now also C4.1; no longer C4.2
Other:
- moved on the sheet: R1, R2, R3, R4, SW1, SW2, SW3, SW4
