File: Electronics/ProtoRev0/BrailleBoy/SolenoidFetMatrix.sch (KiCad schematic (older format))
At the start: 40 parts

Commit message: Added some annotations to make things rather professional :)
Parts:
- renumbered C16 to C14, C17 to C15, C18 to C16, C19 to C17
Connections:
- no-connect marks 0 -> 1
Changed lines of the file:
@@
 encoding utf-8
 Sheet 4 5
-Title ""
-Date ""
-Rev ""
-Comp ""
+Title "Solenoid Matrix and Power Electronics"
+Date "2018-08-07"
+Rev "1.0.0"
+Comp "Devyash Lodha"
 Comment1 ""
 Comment2 ""
@@
 Text Label 5100 4550 0    50   ~ 0
 BotRight
-Text HLabel 5450 2950 2    50   Input ~ 0
+Text HLabel 5100 5350 2    50   Input ~ 0
 PWR_IN
-Text HLabel 5850 4400 0    50   Input ~ 0
+Text HLabel 5100 5450 2    50   Input ~ 0
 GND
 Text HLabel 8950 1250 1    50   Input ~ 0
@@
 GND
 $Comp
-L Device:C C17
+L Device:C C15
 U 1 1 5BDDCF7F
 P 8800 1500
-F 0 "C17" H 8915 1546 50  0000 L CNN
+F 0 "C15" H 8915 1546 50  0000 L CNN
 F 1 "10uF" H 8850 1400 50  0000 L CNN
 F 2 "Capacitors_SMD:C_0805" H 8838 1350 50  0001 C CNN
@@
 $EndComp
 $Comp
-L Device:C C18
+L Device:C C16
 U 1 1 5BDDD0D5
 P 9100 1500
-F 0 "C18" H 9215 1546 50  0000 L CNN
+F 0 "C16" H 9215 1546 50  0000 L CNN
 F 1 "0.1uF" H 9150 1400 50  0000 L CNN
 F 2 "Capacitors_SMD:C_0805" H 9138 1350 50  0001 C CNN
@@
 $EndComp
 $Comp
-L Device:C C16
+L Device:C C14
 U 1 1 5BDDD165
 P 8500 1500
-F 0 "C16" H 8615 1546 50  0000 L CNN
+F 0 "C14" H 8615 1546 50  0000 L CNN
 F 1 "22uF" H 8550 1400 50  0000 L CNN
 F 2 "Capacitors_SMD:C_0805" H 8538 1350 50  0001 C CNN
@@
 $EndComp
 $Comp
-L Device:C C19
+L Device:C C17
 U 1 1 5BDDD1F5
 P 9400 1500
-F 0 "C19" H 9515 1546 50  0000 L CNN
+F 0 "C17" H 9515 1546 50  0000 L CNN
 F 1 "0.1uF" H 9450 1400 50  0000 L CNN
 F 2 "Capacitors_SMD:C_0805" H 9438 1350 50  0001 C CNN
@@
 F24 "MOS_HIGH4" I R 5000 4450 50
 F25 "MOS_HIGH5" I R 5000 4550 50
+F26 "POWER_IN" I R 5000 5350 50
+F27 "GROUND_IN" I R 5000 5450 50
+F28 "DRIVER_VOLTAGE_OUT" I R 5000 5550 50
 $EndSheet
+Wire Wire Line
+	5100 4050 5000 4050
+Wire Wire Line
+	5000 4150 5100 4150
+Wire Wire Line
+	5100 4250 5000 4250
+Wire Wire Line
+	5000 4350 5100 4350
+Wire Wire Line
+	5100 4450 5000 4450
+Wire Wire Line
+	5000 4550 5100 4550
+Wire Wire Line
+	5100 4650 5000 4650
+Wire Wire Line
+	5000 4750 5100 4750
+Wire Wire Line
+	5100 4850 5000 4850
+Wire Wire Line
+	5000 4950 5100 4950
+Wire Wire Line
+	5000 5050 5100 5050
+Wire Wire Line
+	5100 5150 5000 5150
+Wire Wire Line
+	3250 5150 3350 5150
+Wire Wire Line
+	3350 5050 3250 5050
+Wire Wire Line
+	3250 4950 3350 4950
+Wire Wire Line
+	3350 4850 3250 4850
+Wire Wire Line
+	3250 4750 3350 4750
+Wire Wire Line
+	3350 4650 3250 4650
+Wire Wire Line
+	3250 4550 3350 4550
+Wire Wire Line
+	3350 4450 3250 4450
+Wire Wire Line
+	3250 4350 3350 4350
+Wire Wire Line
+	3350 4250 3250 4250
+Wire Wire Line
+	3250 4150 3350 4150
+Wire Wire Line
+	3350 4050 3250 4050
+Wire Wire Line
+	5000 5350 5100 5350
+Wire Wire Line
+	5100 5450 5000 5450
+NoConn ~ 5000 5550
 $EndSCHEMATC

Commit message: Made the schematic sheets a bit prettier
Other:
- note added: "INPUTS/OUTPUTS"
Changed lines of the file:
@@
 Text Notes 3650 800  0    50   ~ 0
 CHARACTER DISPLAY\nDOT_COM = [TOP/MID/BOT][LEFT/RIGHT]\nCHAR_COM = [CHAR[0:5]]
-Text HLabel 3250 4650 0    50   Input ~ 0
+Text HLabel 950  3700 0    50   Input ~ 0
 LOW0
-Text HLabel 3250 4750 0    50   Input ~ 0
+Text HLabel 950  3800 0    50   Input ~ 0
 LOW1
-Text HLabel 3250 4850 0    50   Input ~ 0
+Text HLabel 950  3900 0    50   Input ~ 0
 LOW2
-Text HLabel 3250 4950 0    50   Input ~ 0
+Text HLabel 950  4000 0    50   Input ~ 0
 LOW3
-Text HLabel 3250 5050 0    50   Input ~ 0
+Text HLabel 950  4100 0    50   Input ~ 0
 LOW4
-Text HLabel 3250 5150 0    50   Input ~ 0
+Text HLabel 950  4200 0    50   Input ~ 0
 LOW5
-Text Label 5100 4650 0    50   ~ 0
+Text Label 2150 3700 0    50   ~ 0
 Char0
-Text Label 5100 4750 0    50   ~ 0
+Text Label 2150 3800 0    50   ~ 0
 Char1
-Text Label 5100 4850 0    50   ~ 0
+Text Label 2150 3900 0    50   ~ 0
 Char2
-Text Label 5100 4950 0    50   ~ 0
+Text Label 2150 4000 0    50   ~ 0
 Char3
-Text Label 5100 5050 0    50   ~ 0
+Text Label 2150 4100 0    50   ~ 0
 Char4
-Text Label 5100 5150 0    50   ~ 0
+Text Label 2150 4200 0    50   ~ 0
 Char5
-Text HLabel 3250 4050 0    50   Input ~ 0
+Text HLabel 950  3100 0    50   Input ~ 0
 High0
-Text HLabel 3250 4150 0    50   Input ~ 0
+Text HLabel 950  3200 0    50   Input ~ 0
 High1
-Text HLabel 3250 4250 0    50   Input ~ 0
+Text HLabel 950  3300 0    50   Input ~ 0
 High2
-Text HLabel 3250 4350 0    50   Input ~ 0
+Text HLabel 950  3400 0    50   Input ~ 0
 High3
-Text HLabel 3250 4450 0    50   Input ~ 0
+Text HLabel 950  3500 0    50   Input ~ 0
 High4
-Text HLabel 3250 4550 0    50   Input ~ 0
+Text HLabel 950  3600 0    50   Input ~ 0
 High5
-Text Label 5100 4050 0    50   ~ 0
+Text Label 2150 3100 0    50   ~ 0
 TopLeft
-Text Label 5100 4150 0    50   ~ 0
+Text Label 2150 3200 0    50   ~ 0
 MidLeft
-Text Label 5100 4250 0    50   ~ 0
+Text Label 2150 3300 0    50   ~ 0
 BotLeft
-Text Label 5100 4350 0    50   ~ 0
+Text Label 2150 3400 0    50   ~ 0
 TopRight
-Text Label 5100 4450 0    50   ~ 0
+Text Label 2150 3500 0    50   ~ 0
 MidRight
-Text Label 5100 4550 0    50   ~ 0
+Text Label 2150 3600 0    50   ~ 0
 BotRight
-Text HLabel 5100 5350 2    50   Input ~ 0
+Text HLabel 2150 4400 2    50   Input ~ 0
 PWR_IN
-Text HLabel 5100 5450 2    50   Input ~ 0
+Text HLabel 2150 4500 2    50   Input ~ 0
 GND
 Text HLabel 8950 1250 1    50   Input ~ 0
@@
 DECOUPLING
 $Sheet
-S 3350 3950 1650 2050
+S 1050 3000 1000 1750
 U 5C1CF809
 F0 "FETs and Drivers" 50
 F1 "FETsDrivers.sch" 50
-F2 "HIGH0" I L 3350 4050 50
-F3 "HIGH1" I L 3350 4150 50
-F4 "HIGH2" I L 3350 4250 50
-F5 "HIGH3" I L 3350 4350 50
-F6 "HIGH4" I L 3350 4450 50
-F7 "HIGH5" I L 3350 4550 50
-F8 "LOW0" I L 3350 4650 50
-F9 "LOW1" I L 3350 4750 50
-F10 "LOW2" I L 3350 4850 50
-F11 "LOW3" I L 3350 4950 50
-F12 "LOW4" I L 3350 5050 50
-F13 "LOW5" I L 3350 5150 50
-F14 "MOS_LOW0" I R 5000 4650 50
-F15 "MOS_LOW1" I R 5000 4750 50
-F16 "MOS_LOW2" I R 5000 4850 50
-F17 "MOS_LOW3" I R 5000 4950 50
-F18 "MOS_LOW4" I R 5000 5050 50
-F19 "MOS_LOW5" I R 5000 5150 50
-F20 "MOS_HIGH0" I R 5000 4050 50
-F21 "MOS_HIGH1" I R 5000 4150 50
-F22 "MOS_HIGH2" I R 5000 4250 50
-F23 "MOS_HIGH3" I R 5000 4350 50
-F24 "MOS_HIGH4" I R 5000 4450 50
-F25 "MOS_HIGH5" I R 5000 4550 50
-F26 "POWER_IN" I R 5000 5350 50
-F27 "GROUND_IN" I R 5000 5450 50
-F28 "DRIVER_VOLTAGE_OUT" I R 5000 5550 50
+F2 "HIGH0" I L 1050 3100 50
+F3 "HIGH1" I L 1050 3200 50
+F4 "HIGH2" I L 1050 3300 50
+F5 "HIGH3" I L 1050 3400 50
+F6 "HIGH4" I L 1050 3500 50
+F7 "HIGH5" I L 1050 3600 50
+F8 "LOW0" I L 1050 3700 50
+F9 "LOW1" I L 1050 3800 50
+F10 "LOW2" I L 1050 3900 50
+F11 "LOW3" I L 1050 4000 50
+F12 "LOW4" I L 1050 4100 50
+F13 "LOW5" I L 1050 4200 50
+F14 "MOS_LOW0" I R 2050 3700 50
+F15 "MOS_LOW1" I R 2050 3800 50
+F16 "MOS_LOW2" I R 2050 3900 50
+F17 "MOS_LOW3" I R 2050 4000 50
+F18 "MOS_LOW4" I R 2050 4100 50
+F19 "MOS_LOW5" I R 2050 4200 50
+F20 "MOS_HIGH0" I R 2050 3100 50
+F21 "MOS_HIGH1" I R 2050 3200 50
+F22 "MOS_HIGH2" I R 2050 3300 50
+F23 "MOS_HIGH3" I R 2050 3400 50
+F24 "MOS_HIGH4" I R 2050 3500 50
+F25 "MOS_HIGH5" I R 2050 3600 50
+F26 "POWER_IN" I R 2050 4400 50
+F27 "GROUND_IN" I R 2050 4500 50
+F28 "DRIVER_VOLTAGE_OUT" I R 2050 4600 50
 $EndSheet
 Wire Wire Line
-	5100 4050 5000 4050
-Wire Wire Line
-	5000 4150 5100 4150
-Wire Wire Line
-	5100 4250 5000 4250
-Wire Wire Line
-	5000 4350 5100 4350
-Wire Wire Line
-	5100 4450 5000 4450
-Wire Wire Line
-	5000 4550 5100 4550
-Wire Wire Line
-	5100 4650 5000 4650
-Wire Wire Line
-	5000 4750 5100 4750
-Wire Wire Line
-	5100 4850 5000 4850
-Wire Wire Line
-	5000 4950 5100 4950
-Wire Wire Line
-	5000 5050 5100 5050
-Wire Wire Line
-	5100 5150 5000 5150
-Wire Wire Line
-	3250 5150 3350 5150
-Wire Wire Line
-	3350 5050 3250 5050
-Wire Wire Line
-	3250 4950 3350 4950
-Wire Wire Line
-	3350 4850 3250 4850
-Wire Wire Line
-	3250 4750 3350 4750
-Wire Wire Line
-	3350 4650 3250 4650
-Wire Wire Line
-	3250 4550 3350 4550
-Wire Wire Line
-	3350 4450 3250 4450
-Wire Wire Line
-	3250 4350 3350 4350
-Wire Wire Line
-	3350 4250 3250 4250
-Wire Wire Line
-	3250 4150 3350 4150
-Wire Wire Line
-	3350 4050 3250 4050
-Wire Wire Line
-	5000 5350 5100 5350
-Wire Wire Line
-	5100 5450 5000 5450
-NoConn ~ 5000 5550
+	2150 3100 2050 3100
+Wire Wire Line
+	2050 3200 2150 3200
+Wire Wire Line
+	2150 3300 2050 3300
+Wire Wire Line
+	2050 3400 2150 3400
+Wire Wire Line
+	2150 3500 2050 3500
+Wire Wire Line
+	2050 3600 2150 3600
+Wire Wire Line
+	2150 3700 2050 3700
+Wire Wire Line
+	2050 3800 2150 3800
+Wire Wire Line
+	2150 3900 2050 3900
+Wire Wire Line
+	2050 4000 2150 4000
+Wire Wire Line
+	2050 4100 2150 4100
+Wire Wire Line
+	2150 4200 2050 4200
+Wire Wire Line
+	950  4200 1050 4200
+Wire Wire Line
+	1050 4100 950  4100
+Wire Wire Line
+	950  4000 1050 4000
+Wire Wire Line
+	1050 3900 950  3900
+Wire Wire Line
+	950  3800 1050 3800
+Wire Wire Line
+	1050 3700 950  3700
+Wire Wire Line
+	950  3600 1050 3600
+Wire Wire Line
+	1050 3500 950  3500
+Wire Wire Line
+	950  3400 1050 3400
+Wire Wire Line
+	1050 3300 950  3300
+Wire Wire Line
+	950  3200 1050 3200
+Wire Wire Line
+	1050 3100 950  3100
+Wire Wire Line
+	2050 4400 2150 4400
+Wire Wire Line
+	2150 4500 2050 4500
+NoConn ~ 2050 4600
+Wire Notes Line
+	550  4900 2550 4900
+Wire Notes Line
+	2550 4900 2550 2850
+Wire Notes Line
+	2550 2850 550  2850
+Wire Notes Line
+	550  2850 550  4900
+Text Notes 1250 2850 0    50   ~ 0
+INPUTS/OUTPUTS
 $EndSCHEMATC
