File: Electronics/ProtoRev0/BrailleBoy/Uart.sch (KiCad schematic (older format))
At the start: 11 parts, among them Q1 SS8050-G, Q2 SS8050-G, U6 FT232RL

Commit message: Added some annotations to make things rather professional :)
Parts:
- renumbered C15 to C13
Changed lines of the file:
@@
 encoding utf-8
 Sheet 3 5
-Title ""
-Date ""
-Rev ""
-Comp ""
+Title "FT232(RL)-based UART programming/communications interface"
+Date "2018-08-07"
+Rev "1.0.0"
+Comp "Devyash Lodha"
 Comment1 ""
 Comment2 ""
@@
 P 3150 2000
 AR Path="/5B72E018" Ref="C?"  Part="1"
-AR Path="/5B72DEC1/5B72E018" Ref="C15"  Part="1"
-F 0 "C15" V 2921 2000 50  0000 C CNN
+AR Path="/5B72DEC1/5B72E018" Ref="C13"  Part="1"
+F 0 "C13" V 2921 2000 50  0000 C CNN
 F 1 "0.1uF" V 3012 2000 50  0000 C CNN
 F 2 "Capacitors_SMD:C_0805" H 3150 2000 50  0001 C CNN

Commit message: Made the schematic sheets a bit prettier
Other:
- note added: "FT232-RL UART CONFIGURATION"
- note added: "POWER RAILS"
- moved on the sheet: C13, D5, D6, Q1, Q2, R18, R19, R20, R21, R22, U6
