File: Electronics/ProtoRev0/BrailleBoy/Uart.sch (KiCad schematic (older format))
At the start: 11 parts, among them Q1 SS8050-G, Q2 SS8050-G, U6 FT232RL

Commit message: Uploading all files to transfer this project to another team who is interested in continuing it
Parts:
- removed U6: FT232RL, Package_SO:SSOP-28_5.3x10.2mm_P0.65mm, symbol Interface_USB:FT232RL
- added U?: FT232RL, Package_SO:SSOP-28_5.3x10.2mm_P0.65mm, symbol Interface_USB:FT232RL
Connections:
- net +3V3: now also U?.4 (VCCIO)
- net GND: now also U?.18 (GND), U?.21 (GND), U?.25 (AGND), U?.7 (GND)
- net RX: now also U?.1 (TXD)
- net TX: now also U?.5 (RXD)
- net USB_DM: now also U?.16 (USBD-)
- net USB_DP: now also U?.15 (USBD+)
- net VBUS: now also U?.20 (VCC)
- net at R18.1: now also U?.17 (3V3OUT)
- net at Q1.2 (E), R20.2: now also U?.2 (DTR)
- net at D5.1 (K): now also U?.22 (CBUS1)
- net at D6.1 (K): now also U?.23 (CBUS0)
- net at Q2.3 (C), R19.2: now also U?.3 (RTS)
Changed lines of the file:
@@
 EESchema Schematic File Version 4
 LIBS:BrailleBoy-cache
-EELAYER 26 0
+EELAYER 29 0
 EELAYER END
 $Descr A4 11693 8268
@@
 Comment4 ""
 $EndDescr
-$Comp
-L Interface_USB:FT232RL U?
-U 1 1 5B72DF76
-P 1900 2100
-AR Path="/5B72DF76" Ref="U?"  Part="1"
-AR Path="/5B72DEC1/5B72DF76" Ref="U6"  Part="1"
-F 0 "U6" H 1900 3278 50  0000 C CNN
-F 1 "FT232RL" H 1850 3200 50  0000 C CNN
-F 2 "Package_SO:SSOP-28_5.3x10.2mm_P0.65mm" H 1900 2100 50  0001 C CNN
-F 3 "http://www.ftdichip.com/Products/ICs/FT232RL.htm" H 1900 2100 50  0001 C CNN
-	1    1900 2100
-	1    0    0    -1
-$EndComp
 Wire Wire Line
 	1000 1800 1100 1800
@@
 Text Notes 1950 650  0    50   ~ 0
 FT232-RL UART CONFIGURATION
+$Comp
+L Interface_USB:FT232RL U?
+U 1 1 5D482DCD
+P 1900 2100
+F 0 "U?" H 1900 3281 50  0000 C CNN
+F 1 "FT232RL" H 1900 3190 50  0000 C CNN
+F 2 "Package_SO:SSOP-28_5.3x10.2mm_P0.65mm" H 1900 2100 50  0001 C CNN
+F 3 "http://www.ftdichip.com/Products/ICs/FT232RL.htm" H 1900 2100 50  0001 C CNN
+	1    1900 2100
+	1    0    0    -1
+$EndComp
 $EndSCHEMATC
