File: Electronics/ProtoRev0/BrailleBoy/powermgmt.sch (KiCad schematic (older format))
At the start: 13 parts, among them J1 USB_B_Micro, J2 Battery, U4 AP2115-SOIC, U5 MCP73832-2-OT

Commit message: Uploading all files to transfer this project to another team who is interested in continuing it
Parts:
- removed U4: AP2115-SOIC, Housings_SOIC:SOIC-8_3.9x4.9mm_Pitch1.27mm, symbol Custom:AP2115-SOIC
- added U?: AP2115-SOIC, symbol Custom:AP2115-SOIC
Connections:
- net +3V3: now also U?.1 (VOUT)
- net +BATT: now also U?.5 (EN), U?.8 (VIN)
- net -BATT: now also U?.6 (GND), U?.7 (GND)
Changed lines of the file:
@@
 EESchema Schematic File Version 4
 LIBS:BrailleBoy-cache
-EELAYER 26 0
+EELAYER 29 0
 EELAYER END
 $Descr A4 11693 8268
@@
 $EndComp
 $Comp
-L Custom:AP2115-SOIC U?
-U 1 1 5B66D9AC
-P 2900 1900
-AR Path="/5B66D9AC" Ref="U?"  Part="1"
-AR Path="/5B66D91B/5B66D9AC" Ref="U4"  Part="1"
-F 0 "U4" H 3200 2075 50  0000 C CNN
-F 1 "AP2115-SOIC" H 3200 1984 50  0000 C CNN
-F 2 "Housings_SOIC:SOIC-8_3.9x4.9mm_Pitch1.27mm" H 2900 2000 50  0001 C CNN
-F 3 "" H 2900 2000 50  0001 C CNN
-	1    2900 1900
-	1    0    0    -1
-$EndComp
-$Comp
 L Connector:USB_B_Micro J?
 U 1 1 5B66D9B3
@@
 Wire Notes Line
 	2100 650  2100 2750
+$Comp
+L Custom:AP2115-SOIC U?
+U 1 1 5D4816D5
+P 2900 1900
+F 0 "U?" H 3200 2075 50  0000 C CNN
+F 1 "AP2115-SOIC" H 3200 1984 50  0000 C CNN
+F 2 "" H 2900 2000 50  0001 C CNN
+F 3 " https://www.mouser.com/datasheet/2/115/AP2115-464923.pdf" H 2900 2000 50  0001 C CNN
+	1    2900 1900
+	1    0    0    -1
+$EndComp
 $EndSCHEMATC
